File: raptor.ups/_saved_raptor.sch (KiCad schematic (older format))
At the start: 9 parts, among them P1 TP4056, P2 CONN_RPI+HUB, P3 CONN_220V

Commit message: Postępy nad schematem...
Parts:
- P3: footprint (none) -> Terminal_Blocks:TerminalBlock_Pheonix_PT-3.5mm_2pol
Changed lines of the file:
@@
 F 0 "P3" H 1600 3000 50  0000 C CNN
 F 1 "CONN_220V" V 1700 2850 50  0000 C CNN
-F 2 "" H 1600 2850 50  0000 C CNN
+F 2 "Terminal_Blocks:TerminalBlock_Pheonix_PT-3.5mm_2pol" H 1600 2850 50  0001 C CNN
 F 3 "" H 1600 2850 50  0000 C CNN
 	1    1600 2850
