File: raptor.ups/raptor.kicad_pcb (KiCad board)
At the start: 2 copper layers, 9 parts, among them P1 TP4056, P2 CONN_RPI+HUB, P3 CONN_220V

Commit message: Płytka prawie gotowa!
Parts:
- removed Z1: Zasilacz, my-poi:GPV-20-5
- added CH1: TP4056, my-poi:TP4056, F.Cu at (112.0, 118.0)
- added P4: Power, my-poi:GPV-20-5, F.Cu at (158.0, 58.0)
- P1: value TP4056 -> CONN_220V; footprint my-poi:TP4056 -> my-poi:TerminalBlock_2pin_5mm
- P2: value CONN_RPI+HUB -> CONN_RPI; footprint Terminal_Blocks:TerminalBlock_Pheonix_PT-3.5mm_2pol -> my-poi:TerminalBlock_2pin_5mm
- P3: value CONN_220V -> CONN_HUB; footprint Terminal_Blocks:TerminalBlock_Pheonix_PT-3.5mm_2pol -> my-poi:TerminalBlock_2pin_5mm
- moved P1 46.1 mm to (82.0, 73.0), turned to 270 degrees
- moved S1 27.7 mm to (111.0, 91.0), turned to 180 degrees
- moved P2 25.0 mm to (82.0, 96.0), turned to 270 degrees
- moved P3 19.0 mm to (82.0, 117.0), turned to 270 degrees
- moved D1 18.1 mm to (143.0, 93.0), turned to 90 degrees
- moved D2 8.94 mm to (137.0, 93.0), turned to 270 degrees
- moved BT1 7.62 mm to (190.0, 112.0)
- moved BT2 4.24 mm to (190.0, 88.0)
Connections:
- D2 pad 2: Net-(D2-Pad2) -> Net-(CH1-Pad3)
- P1 pad 1: VCC -> Net-(P1-Pad1)
- P1 pad 2: GND -> Net-(P1-Pad2)
- P3 pad 1: Net-(P3-Pad1) -> Net-(P2-Pad1)
- P3 pad 2: Net-(P3-Pad2) -> GND
Routing:
- net GND: track 60.7 -> 153.3 mm
- net Net-(BT1-Pad1): track 0.00 -> 68.1 mm
- net Net-(BT1-Pad2): track 0.00 -> 55.0 mm
- net Net-(D1-Pad1): track 70.8 -> 15.9 mm
- net VCC: track 26.1 -> 60.5 mm
- net Net-(P1-Pad1): track 0.00 -> 33.6 mm
- net Net-(P3-Pad1): track 33.3 -> 0.00 mm
- net Net-(P3-Pad2): track 27.3 -> 0.00 mm
- net Net-(P2-Pad1): track 17.5 -> 32.8 mm
- net Net-(P1-Pad2): track 0.00 -> 14.4 mm
- net Net-(CH1-Pad3): track 0.00 -> 11.1 mm

Commit message: Jeszcze poprawki płytki PCB UPS-a.
Parts:
- moved CH1 5.00 mm to (117.0, 118.0)
- moved S1 3.16 mm to (112.0, 94.0)
- moved BT1 2.24 mm to (192.0, 111.0)
- moved P2 2.24 mm to (83.0, 94.0)
- moved BT2 2.00 mm to (192.0, 88.0)
- moved D1 2.00 mm to (145.0, 93.0)
- moved P4 2.00 mm to (160.0, 58.0)
- moved D2 1.00 mm to (138.0, 93.0)
- moved P1 1.00 mm to (82.0, 72.0)
- moved P3 1.00 mm to (83.0, 117.0)
Connections:
- P2 pad 1: Net-(P2-Pad1) -> GND
- P2 pad 2: GND -> Net-(P2-Pad2)
- P3 pad 1: Net-(P2-Pad1) -> Net-(P2-Pad2)
- S1 pad 3: Net-(P2-Pad1) -> Net-(P2-Pad2)
Routing:
- net Net-(P2-Pad1): track 32.8 -> 0.00 mm
- net Net-(P2-Pad2): track 0.00 -> 29.1 mm
- net Net-(BT1-Pad1): track 68.1 -> 59.6 mm
- net Net-(P1-Pad1): track 33.6 -> 41.7 mm
- net Net-(D1-Pad1): track 15.9 -> 19.9 mm
- net Net-(CH1-Pad3): track 11.1 -> 7.44 mm
- net Net-(BT1-Pad2): track 55.0 -> 51.6 mm
- net GND: track 153.3 -> 155.9 mm
- net VCC: track 60.5 -> 58.1 mm
- net Net-(P1-Pad2): track 14.4 -> 16.0 mm

Commit message: Praktycznie gotowa PCB UPS-a.
Parts:
- moved BT1 6.00 mm to (192.0, 117.0)
- moved BT2 6.00 mm to (192.0, 94.0)
- moved D1 1.00 mm to (144.0, 93.0)
Routing:
- net GND: track 155.9 -> 0.00 mm
- net Net-(BT1-Pad1): track 59.6 -> 53.6 mm
- net Net-(BT1-Pad2): track 51.6 -> 48.3 mm
- net VCC: track 58.1 -> 57.1 mm
- net Net-(D1-Pad1): track 19.9 -> 18.9 mm
- added copper zone on B.Cu, net GND
