File: raptor.ups/raptor.sch (KiCad schematic (older format))
At the start: 9 parts, among them P1 TP4056, P2 CONN_RPI+HUB, P3 CONN_220V

Commit message: Pierwsze ścieżki :)
Parts:
- BT1, BT2: footprint (none) -> my-poi:18650
- P1: footprint (none) -> my-poi:TP4056
- P3: footprint (none) -> Terminal_Blocks:TerminalBlock_Pheonix_PT-3.5mm_2pol
- S1: footprint (none) -> my-poi:STEP-UP
Changed lines of the file:
@@
 F 0 "P1" H 5600 3100 60  0000 C CNN
 F 1 "TP4056" V 5600 2750 60  0000 C CNN
-F 2 "" H 5600 3450 60  0001 C CNN
+F 2 "my-poi:TP4056" H 5600 3450 60  0001 C CNN
 F 3 "" H 5600 3450 60  0000 C CNN
 	1    5600 2900
@@
 F 0 "BT1" H 6950 2950 50  0000 L CNN
 F 1 "18650" H 6950 2850 50  0000 L CNN
-F 2 "" V 6850 2940 50  0001 C CNN
+F 2 "my-poi:18650" V 6850 2940 50  0001 C CNN
 F 3 "" V 6850 2940 50  0000 C CNN
 	1    6850 2900
@@
 F 0 "BT2" H 7450 2950 50  0000 L CNN
 F 1 "18650" H 7450 2850 50  0000 L CNN
-F 2 "" V 7350 2940 50  0001 C CNN
+F 2 "my-poi:18650" V 7350 2940 50  0001 C CNN
 F 3 "" V 7350 2940 50  0000 C CNN
 	1    7350 2900
@@
 F 0 "S1" H 8900 2450 60  0000 C CNN
 F 1 "STEP-UP" V 8900 2150 60  0000 C CNN
-F 2 "" H 8900 2500 60  0001 C CNN
+F 2 "my-poi:STEP-UP" H 8900 2500 60  0001 C CNN
 F 3 "" H 8900 2500 60  0000 C CNN
 	1    8900 2500
@@
 F 0 "P3" H 1600 3000 50  0000 C CNN
 F 1 "CONN_220V" V 1700 2850 50  0000 C CNN
-F 2 "" H 1600 2850 50  0000 C CNN
+F 2 "Terminal_Blocks:TerminalBlock_Pheonix_PT-3.5mm_2pol" H 1600 2850 50  0001 C CNN
 F 3 "" H 1600 2850 50  0000 C CNN
 	1    1600 2850

Commit message: Płytka prawie gotowa!
Parts:
- removed P1: TP4056, my-poi:TP4056, symbol TP4056
- removed Z1: Zasilacz, my-poi:GPV-20-5, symbol Zasilacz
- added CH1: TP4056, my-poi:TP4056, symbol TP4056
- added P3: CONN_HUB, my-poi:TerminalBlock_2pin_5mm, symbol CONN_01X02
- added P4: Power, my-poi:GPV-20-5, symbol Power
- P1: renamed from P3; footprint Terminal_Blocks:TerminalBlock_Pheonix_PT-3.5mm_2pol -> my-poi:TerminalBlock_2pin_5mm
- P2: value CONN_RPI+HUB -> CONN_RPI; footprint Terminal_Blocks:TerminalBlock_Pheonix_PT-3.5mm_2pol -> my-poi:TerminalBlock_2pin_5mm
Connections:
- net GND: now also CH1.2 (-), CH1.6 (OUT-), P3.2 (P2), P4.4 (V-(BLACK))
- net VCC: now also CH1.1 (+), P4.3 (V+(RED))
- net at D2.2 (A): now also CH1.3 (OUT+)
- net at BT1.1, BT2.1: now also CH1.4 (B+)
- net at BT1.2, BT2.2: now also CH1.5 (B-)
- net at P2.1 (P1), S1.3 (OUT+): now also P3.1 (P1)
- net at P1.1 (P1): now also P4.2 (AC/N(BLUE))
- net at P1.2 (P2): now also P4.1 (AC/L(BROWN))
Changed lines of the file:
@@
 $EndComp
-$Comp
-L TP4056 P1
-U 1 1 5738EA09
-P 5600 2900
-F 0 "P1" H 5600 3100 60  0000 C CNN
-F 1 "TP4056" V 5600 2750 60  0000 C CNN
-F 2 "my-poi:TP4056" H 5600 3450 60  0001 C CNN
-F 3 "" H 5600 3450 60  0000 C CNN
-	1    5600 2900
-	1    0    0    -1
-$EndComp
-Wire Wire Line
-	5000 1950 5000 2600
-Wire Wire Line
-	5000 2600 5150 2600
 $Comp
 L GND #PWR07
@@
 	1    0    0    -1
 $EndComp
-Wire Wire Line
-	5150 3200 5000 3200
-Wire Wire Line
-	6100 3200 6250 3200
 $Comp
 L Battery BT1
@@
 	1    0    0    -1
 $EndComp
-Wire Wire Line
-	6850 2750 6850 2700
-Wire Wire Line
-	6350 2700 7350 2700
-Wire Wire Line
-	6350 2700 6350 2800
-Wire Wire Line
-	6350 2800 6100 2800
-Wire Wire Line
-	6100 3000 6350 3000
-Wire Wire Line
-	6350 3000 6350 3100
-Wire Wire Line
-	6350 3100 7350 3100
-Wire Wire Line
-	6850 3100 6850 3050
-Wire Wire Line
-	7350 2700 7350 2750
-Connection ~ 6850 2700
-Wire Wire Line
-	7350 3100 7350 3050
-Connection ~ 6850 3100
 $Comp
 L D D2
@@
 	0    -1   -1   0
 $EndComp
-Wire Wire Line
-	6100 2600 7800 2600
-Wire Wire Line
-	8100 2600 8400 2600
-Wire Wire Line
-	8250 2600 8250 2450
-Wire Wire Line
-	8250 1950 8250 2150
-$Comp
-L STEP-UP S1
-U 1 1 573A18DA
-P 8900 2500
-F 0 "S1" H 8900 2450 60  0000 C CNN
-F 1 "STEP-UP" V 8900 2150 60  0000 C CNN
-F 2 "my-poi:STEP-UP" H 8900 2500 60  0001 C CNN
-F 3 "" H 8900 2500 60  0000 C CNN
-	1    8900 2500
-	1    0    0    -1
-$EndComp
-Wire Wire Line
-	5000 3200 5000 3600
-Wire Wire Line
-	6250 3200 6250 3600
 $Comp
 L GND #PWR09
@@
 	1    0    0    -1
 $EndComp
-Connection ~ 8250 2600
-Wire Wire Line
-	8400 3050 8250 3050
-Wire Wire Line
-	8250 3050 8250 3600
-Wire Wire Line
-	9400 3050 9550 3050
-Wire Wire Line
-	9550 3050 9550 3600
 $Comp
 L CONN_01X02 P2
@@
 P 10300 2650
 F 0 "P2" H 10300 2800 50  0000 C CNN
-F 1 "CONN_RPI+HUB" V 10400 2650 50  0000 C CNN
-F 2 "Terminal_Blocks:TerminalBlock_Pheonix_PT-3.5mm_2pol" H 10300 2650 50  0001 C CNN
+F 1 "CONN_RPI" V 10400 2650 50  0000 C CNN
+F 2 "my-poi:TerminalBlock_2pin_5mm" H 10300 2650 50  0001 C CNN
 F 3 "" H 10300 2650 50  0000 C CNN
 	1    10300 2650
 	1    0    0    -1
 $EndComp
-Wire Wire Line
-	9400 2600 10100 2600
-Wire Wire Line
-	10100 2700 9950 2700
-Wire Wire Line
-	9950 2700 9950 3600
-$Comp
-L Zasilacz Z1
-U 1 1 573A5D6C
+$Comp
+L CONN_01X02 P1
+U 1 1 573A2ACA
+P 1600 2850
+F 0 "P1" H 1600 3000 50  0000 C CNN
+F 1 "CONN_220V" V 1700 2850 50  0000 C CNN
+F 2 "my-poi:TerminalBlock_2pin_5mm" H 1600 2850 50  0001 C CNN
+F 3 "" H 1600 2850 50  0000 C CNN
+	1    1600 2850
+	-1   0    0    1
+$EndComp
+$Comp
+L Power P4
+U 1 1 573CA8A3
 P 3800 2650
-F 0 "Z1" H 3400 2400 60  0000 C CNN
-F 1 "Zasilacz" H 3850 2400 60  0000 C CNN
+F 0 "P4" H 3400 2400 60  0000 C CNN
+F 1 "Power" H 3850 2400 60  0000 C CNN
 F 2 "my-poi:GPV-20-5" H 3800 2650 60  0001 C CNN
 F 3 "" H 3800 2650 60  0000 C CNN
@@
 	1    0    0    -1
 $EndComp
+$Comp
+L TP4056 CH1
+U 1 1 573CB3D3
+P 5600 2900
+F 0 "CH1" H 5600 3100 60  0000 C CNN
+F 1 "TP4056" V 5600 2850 60  0000 C CNN
+F 2 "my-poi:TP4056" H 5600 3450 60  0001 C CNN
+F 3 "" H 5600 3450 60  0000 C CNN
+	1    5600 2900
+	1    0    0    -1
+$EndComp
+$Comp
+L STEP-UP S1
+U 1 1 573CB83C
+P 8900 2500
+F 0 "S1" H 8850 2450 60  0000 C CNN
+F 1 "STEP-UP" V 8850 2150 60  0000 C CNN
+F 2 "my-poi:STEP-UP" H 8850 2500 60  0001 C CNN
+F 3 "" H 8850 2500 60  0000 C CNN
+	1    8900 2500
+	1    0    0    -1
+$EndComp
+$Comp
+L CONN_01X02 P3
+U 1 1 573CBE19
+P 10300 3150
+F 0 "P3" H 10300 3300 50  0000 C CNN
+F 1 "CONN_HUB" V 10400 3150 50  0000 C CNN
+F 2 "my-poi:TerminalBlock_2pin_5mm" H 10300 3150 50  0001 C CNN
+F 3 "" H 10300 3150 50  0000 C CNN
+	1    10300 3150
+	1    0    0    -1
+$EndComp
+Wire Wire Line
+	5000 1950 5000 2600
+Wire Wire Line
+	5000 2600 5150 2600
+Wire Wire Line
+	5150 3200 5000 3200
+Wire Wire Line
+	6100 3200 6250 3200
+Wire Wire Line
+	6850 2750 6850 2700
+Wire Wire Line
+	6350 2700 7350 2700
+Wire Wire Line
+	6350 2700 6350 2800
+Wire Wire Line
+	6350 2800 6100 2800
+Wire Wire Line
+	6100 3000 6350 3000
+Wire Wire Line
+	6350 3000 6350 3100
+Wire Wire Line
+	6350 3100 7350 3100
+Wire Wire Line
+	6850 3100 6850 3050
+Wire Wire Line
+	7350 2700 7350 2750
+Connection ~ 6850 2700
+Wire Wire Line
+	7350 3100 7350 3050
+Connection ~ 6850 3100
+Wire Wire Line
+	6100 2600 7800 2600
+Wire Wire Line
+	8100 2600 8400 2600
+Wire Wire Line
+	8250 2600 8250 2450
+Wire Wire Line
+	8250 1950 8250 2150
+Wire Wire Line
+	5000 3200 5000 3600
+Wire Wire Line
+	6250 3200 6250 3600
+Connection ~ 8250 2600
+Wire Wire Line
+	8400 3050 8250 3050
+Wire Wire Line
+	8250 3050 8250 3600
+Wire Wire Line
+	9400 3050 9550 3050
+Wire Wire Line
+	9550 3050 9550 3600
+Wire Wire Line
+	9400 2600 10100 2600
 Wire Wire Line
 	4600 1950 4600 2800
@@
 Wire Wire Line
 	4600 3000 4450 3000
-$Comp
-L CONN_01X02 P3
-U 1 1 573A2ACA
-P 1600 2850
-F 0 "P3" H 1600 3000 50  0000 C CNN
-F 1 "CONN_220V" V 1700 2850 50  0000 C CNN
-F 2 "Terminal_Blocks:TerminalBlock_Pheonix_PT-3.5mm_2pol" H 1600 2850 50  0001 C CNN
-F 3 "" H 1600 2850 50  0000 C CNN
-	1    1600 2850
-	-1   0    0    1
-$EndComp
 Wire Wire Line
 	3000 2800 1800 2800
@@
 	2000 3000 2050 3000
 Connection ~ 2050 3000
+Wire Wire Line
+	9950 3600 9950 2700
+Wire Wire Line
+	9950 2700 10100 2700
+Wire Wire Line
+	10100 3200 9950 3200
+Connection ~ 9950 3200
+Wire Wire Line
+	10100 3100 9800 3100
+Wire Wire Line
+	9800 3100 9800 2600
+Connection ~ 9800 2600
 $EndSCHEMATC

Commit message: Jeszcze poprawki płytki PCB UPS-a.
Connections:
- net GND: now also P2.1 (P1); no longer P2.2 (P2)
- net at P3.1 (P1), S1.3 (OUT+): now also P2.2 (P2); no longer P2.1 (P1)
Other:
- moved on the sheet: P2
Changed lines of the file:
@@
 L CONN_01X02 P2
 U 1 1 573A2AD6
-P 10300 2650
-F 0 "P2" H 10300 2800 50  0000 C CNN
-F 1 "CONN_RPI" V 10400 2650 50  0000 C CNN
-F 2 "my-poi:TerminalBlock_2pin_5mm" H 10300 2650 50  0001 C CNN
-F 3 "" H 10300 2650 50  0000 C CNN
-	1    10300 2650
+P 10300 2550
+F 0 "P2" H 10300 2700 50  0000 C CNN
+F 1 "CONN_RPI" V 10400 2550 50  0000 C CNN
+F 2 "my-poi:TerminalBlock_2pin_5mm" H 10300 2550 50  0001 C CNN
+F 3 "" H 10300 2550 50  0000 C CNN
+	1    10300 2550
 	1    0    0    -1
 $EndComp
@@
 Connection ~ 2050 3000
 Wire Wire Line
-	9950 3600 9950 2700
-Wire Wire Line
-	9950 2700 10100 2700
-Wire Wire Line
 	10100 3200 9950 3200
 Connection ~ 9950 3200
@@
 	9800 3100 9800 2600
 Connection ~ 9800 2600
+Wire Wire Line
+	9950 3600 9950 2500
+Wire Wire Line
+	9950 2500 10100 2500
 $EndSCHEMATC
