File: raptor.cam/camera.sch (KiCad schematic (older format))
At the start: 2 parts, among them P1 CONN_01X15, P2 FFC_FPC_connector_01X15

Commit message: Prace nad płytką
Parts:
- removed P2: FFC_FPC_connector_01X15, rpi:FFC_connector_15x1.0mm, symbol CONN_01X15
- added P2: CONN_01X05, Pin_Headers:Pin_Header_Straight_1x05_Pitch2.54mm, symbol CONN_01X05
- added P3: CONN_01X16, objects:flat_cable_connector_16pin, symbol CONN_01X16
- P1: footprint rpi:flat_cable_connector_15pin -> objects:FFC_connector_15x1.0mm
Connections:
- wire segments 15 -> 33
Changed lines of the file:
@@
 EESchema Schematic File Version 2
+LIBS:camera-cache
 LIBS:power
 LIBS:device
@@
 LIBS:contrib
 LIBS:valves
-LIBS:camera-cache
 EELAYER 25 0
 EELAYER END
@@
 encoding utf-8
 Sheet 1 1
-Title ""
+Title "Raptor"
 Date ""
 Rev ""
@@
 $EndDescr
 $Comp
-L CONN_01X15 P2
-U 1 1 58C3C235
-P 4750 3150
-F 0 "P2" H 4750 3950 50  0000 C CNN
-F 1 "FFC_FPC_connector_01X15" V 4850 3150 50  0000 C CNN
-F 2 "rpi:FFC_connector_15x1.0mm" V 4950 3150 50  0000 C CNN
-F 3 "" H 4750 3150 50  0000 C CNN
-	1    4750 3150
+L CONN_01X05 P2
+U 1 1 58DDF822
+P 7300 3200
+F 0 "P2" H 7300 3500 50  0000 C CNN
+F 1 "CONN_01X05" V 7400 3200 50  0000 C CNN
+F 2 "Pin_Headers:Pin_Header_Straight_1x05_Pitch2.54mm" H 7300 3200 50  0000 C CNN
+F 3 "" H 7300 3200 50  0000 C CNN
+	1    7300 3200
 	1    0    0    -1
 $EndComp
 $Comp
 L CONN_01X15 P1
-U 1 1 58C3C2CF
-P 3550 3150
-F 0 "P1" H 3550 3950 50  0000 C CNN
-F 1 "CONN_01X15" V 3650 3150 50  0000 C CNN
-F 2 "rpi:flat_cable_connector_15pin" V 3750 3150 50  0000 C CNN
-F 3 "" H 3550 3150 50  0000 C CNN
-	1    3550 3150
-	-1   0    0    -1
+U 1 1 58DDF909
+P 5900 4300
+F 0 "P1" V 5200 4100 50  0000 C CNN
+F 1 "CONN_01X15" H 6000 4000 50  0000 C CNN
+F 2 "objects:FFC_connector_15x1.0mm" V 6000 4100 50  0000 C CNN
+F 3 "" V 6000 4100 50  0000 C CNN
+	1    5900 4300
+	1    0    0    -1
+$EndComp
+$Comp
+L CONN_01X16 P3
+U 1 1 58DE03D8
+P 6000 2700
+F 0 "P3" V 5200 2900 50  0000 C CNN
+F 1 "CONN_01X16" H 6000 3000 50  0000 C CNN
+F 2 "objects:flat_cable_connector_16pin" V 6000 2900 50  0000 C CNN
+F 3 "" V 6000 2900 50  0000 C CNN
+	1    6000 2700
+	1    0    0    -1
 $EndComp
 Wire Wire Line
-	3750 2450 4550 2450
+	5300 4300 5300 2700
 Wire Wire Line
-	3750 2550 4550 2550
+	5400 4300 5400 2700
 Wire Wire Line
-	3750 2650 4550 2650
+	5500 4300 5500 2700
 Wire Wire Line
-	3750 2750 4550 2750
+	5600 4300 5600 2700
 Wire Wire Line
-	3750 2850 4550 2850
+	5700 4300 5700 2700
 Wire Wire Line
-	3750 2950 4550 2950
+	5900 4300 5900 4200
 Wire Wire Line
-	3750 3050 4550 3050
+	5900 4200 5800 4200
 Wire Wire Line
-	3750 3150 4550 3150
+	5800 4200 5800 2700
 Wire Wire Line
-	3750 3250 4550 3250
+	6000 4300 6000 4100
 Wire Wire Line
-	3750 3350 4550 3350
+	6000 4100 5900 4100
 Wire Wire Line
-	3750 3450 4550 3450
+	5900 4100 5900 2700
 Wire Wire Line
-	3750 3550 4550 3550
+	6200 4300 6200 4000
 Wire Wire Line
-	3750 3650 4550 3650
+	6200 4000 6000 4000
 Wire Wire Line
-	3750 3750 4550 3750
+	6000 4000 6000 2700
 Wire Wire Line
-	3750 3850 4550 3850
+	6300 4300 6300 3900
+Wire Wire Line
+	6300 3900 6100 3900
+Wire Wire Line
+	6100 3900 6100 2700
+Wire Wire Line
+	6500 4300 6500 3800
+Wire Wire Line
+	6500 3800 6200 3800
+Wire Wire Line
+	6200 3800 6200 2700
+Wire Wire Line
+	6600 4300 6600 3700
+Wire Wire Line
+	6600 3700 6300 3700
+Wire Wire Line
+	6300 3700 6300 2700
+Wire Wire Line
+	6400 2700 6400 3400
+Wire Wire Line
+	6400 3400 7100 3400
+Wire Wire Line
+	6500 2700 6500 3300
+Wire Wire Line
+	6500 3300 7100 3300
+Wire Wire Line
+	6600 2700 6600 3200
+Wire Wire Line
+	6600 3200 7100 3200
+Wire Wire Line
+	6700 2700 6700 3100
+Wire Wire Line
+	6700 3100 7100 3100
+Wire Wire Line
+	6800 2700 6800 3000
+Wire Wire Line
+	6800 3000 7100 3000
 $EndSCHEMATC
