File: raptor.cam/camera.kicad_pcb (KiCad board)
At the start: 2 copper layers, 2 parts, among them P1 CONN_01X15, P2 FFC_FPC_connector_01X15

Commit message: Kamera cd.
Parts:
- removed P2: FFC_FPC_connector_01X15, rpi:FFC_connector_15x1.0mm
- added ?: , rpi:FFC_connector_15x1.0mm, F.Cu at (148.0, 115.6)
- added ?: , rpi:2.20mmDrill, F.Cu at (137.6, 122.0)
- added ?: , rpi:2.20mmDrill, F.Cu at (158.5, 109.5)
- added ?: , rpi:2.20mmDrill, F.Cu at (158.5, 122.0)
- added ?: , rpi:2.20mmDrill, F.Cu at (137.5, 109.5)
- ?: renamed from P1; value CONN_01X15 -> (none)
Other:
- board outline added: 25 x 25 mm

Commit message: Korekta płytki adaptera kamery
Parts:
- moved ? 1.10 mm to (148.0, 104.0)
- moved ? 0.05 mm to (158.5, 109.5)
- moved ? 0.05 mm to (158.5, 122.0)
- moved ? 0.05 mm to (137.5, 109.5)
Routing:
- net Net-(P1-Pad8): track 11.1 -> 12.3 mm
- net Net-(P1-Pad5): track 9.63 -> 10.8 mm
- net Net-(P1-Pad3): track 10.0 -> 11.2 mm
- net Net-(P1-Pad4): track 11.8 -> 13.0 mm
- net Net-(P1-Pad7): track 9.21 -> 10.4 mm
- net Net-(P1-Pad6): track 11.4 -> 12.6 mm
- net Net-(P1-Pad2): track 12.3 -> 13.5 mm
- net Net-(P1-Pad1): track 10.5 -> 11.7 mm
- net Net-(P1-Pad9): track 9.27 -> 10.4 mm
- net Net-(P1-Pad13): track 10.1 -> 11.2 mm
- net Net-(P1-Pad12): track 11.9 -> 13.0 mm
- net Net-(P1-Pad11): track 9.69 -> 10.8 mm
- net Net-(P1-Pad10): track 11.5 -> 12.6 mm
- net Net-(P1-Pad14): track 12.3 -> 13.4 mm
- net Net-(P1-Pad15): track 10.5 -> 11.6 mm
Other:
- board text added: "Raptor"

Commit message: Przesunąłem złącze FFC od otworów.
Parts:
- moved ? 0.40 mm to (148.0, 115.2)
Changed lines of the file:
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@@
     (links 15)
     (no_connects 0)
-    (area 135.419999 98.874999 160.620001 124.100001)
+    (area 121.920001 89.421833 174.22 132.100001)
     (thickness 1.6)
     (drawings 10)
-    (tracks 48)
+    (tracks 51)
     (zones 0)
     (modules 6)
@@
   )
   (module rpi:FFC_connector_15x1.0mm (layer F.Cu)
-    (at 147.97 115.6)
+    (at 147.97 115.2)
     (descr "Molex Panelmate series connector, 1.25mm pitch, side entry SMT, P/N: 53780-1570")
     (tags "conn molex panelmate")
@@
   (gr_line (start 135.52 124) (end 135.52 99) (angle 90) (layer Edge.Cuts) (width 0.2))
   (gr_line (start 160.52 124) (end 135.52 124) (angle 90) (layer Edge.Cuts) (width 0.2))
-  (segment (start 143.07 113.16) (end 143.07 106.6) (width 0.25) (layer F.Cu) (net 1))
-  (segment (start 140.5311 104.0611) (end 140.5311 102.9936) (width 0.25) (layer F.Cu) (net 1))
-  (segment (start 143.07 106.6) (end 140.5311 104.0611) (width 0.25) (layer F.Cu) (net 1))
-  (segment (start 144.07 113.16) (end 144.07 106.6) (width 0.25) (layer F.Cu) (net 2))
-  (segment (start 142.0311 104.5611) (end 142.0311 100.9936) (width 0.25) (layer F.Cu) (net 2))
-  (segment (start 144.07 106.6) (end 142.0311 104.5611) (width 0.25) (layer F.Cu) (net 2))
-  (segment (start 145.07 113.16) (end 145.07 106.6) (width 0.25) (layer F.Cu) (net 3))
-  (segment (start 143.5311 105.0611) (end 143.5311 102.9936) (width 0.25) (layer F.Cu) (net 3))
-  (segment (start 145.07 106.6) (end 143.5311 105.0611) (width 0.25) (layer F.Cu) (net 3))
-  (segment (start 146.07 113.16) (end 146.07 106.6) (width 0.25) (layer F.Cu) (net 4))
-  (segment (start 145.0311 105.5611) (end 145.0311 100.9936) (width 0.25) (layer F.Cu) (net 4))
-  (segment (start 146.07 106.6) (end 145.0311 105.5611) (width 0.25) (layer F.Cu) (net 4))
-  (segment (start 147.07 113.16) (end 147.07 106.6) (width 0.25) (layer F.Cu) (net 5))
-  (segment (start 146.5311 106.0611) (end 146.5311 102.9936) (width 0.25) (layer F.Cu) (net 5))
-  (segment (start 147.07 106.6) (end 146.5311 106.0611) (width 0.25) (layer F.Cu) (net 5))
-  (segment (start 148.07 113.16) (end 148.07 101.0325) (width 0.25) (layer F.Cu) (net 6))
+  (segment (start 143.07 112.76) (end 143.07 106.5) (width 0.25) (layer F.Cu) (net 1) (status 400000))
+  (segment (start 140.5311 103.9611) (end 140.5311 102.9936) (width 0.25) (layer F.Cu) (net 1) (status 800000))
+  (segment (start 143.07 106.5) (end 140.5311 103.9611) (width 0.25) (layer F.Cu) (net 1))
+  (segment (start 144.07 112.76) (end 144.07 106.5) (width 0.25) (layer F.Cu) (net 2) (status 400000))
+  (segment (start 142.0311 104.4611) (end 142.0311 100.9936) (width 0.25) (layer F.Cu) (net 2) (status 800000))
+  (segment (start 144.07 106.5) (end 142.0311 104.4611) (width 0.25) (layer F.Cu) (net 2))
+  (segment (start 145.07 112.76) (end 145.07 106.5) (width 0.25) (layer F.Cu) (net 3) (status 400000))
+  (segment (start 143.5311 104.9611) (end 143.5311 102.9936) (width 0.25) (layer F.Cu) (net 3) (status 800000))
+  (segment (start 145.07 106.5) (end 143.5311 104.9611) (width 0.25) (layer F.Cu) (net 3))
+  (segment (start 146.07 112.76) (end 146.07 106.5) (width 0.25) (layer F.Cu) (net 4) (status 400000))
+  (segment (start 145.0311 105.4611) (end 145.0311 100.9936) (width 0.25) (layer F.Cu) (net 4) (status 800000))
+  (segment (start 146.07 106.5) (end 145.0311 105.4611) (width 0.25) (layer F.Cu) (net 4))
+  (segment (start 147.07 112.76) (end 147.07 106.5) (width 0.25) (layer F.Cu) (net 5) (status 400000))
+  (segment (start 146.5311 105.9611) (end 146.5311 102.9936) (width 0.25) (layer F.Cu) (net 5) (status 800000))
+  (segment (start 147.07 106.5) (end 146.5311 105.9611) (width 0.25) (layer F.Cu) (net 5))
+  (segment (start 148.07 112.76) (end 148.07 101.0325) (width 0.25) (layer F.Cu) (net 6) (status C00000))
+  (segment (start 148.07 101.0325) (end 148.0311 100.9936) (width 0.25) (layer F.Cu) (net 6) (status C00000))
   (segment (start 148.07 101.0325) (end 148.0311 100.9936) (width 0.25) (layer F.Cu) (net 6))
   (segment (start 147.96 101.0647) (end 148.0311 100.9936) (width 0.25) (layer F.Cu) (net 6))
-  (segment (start 149.07 113.16) (end 149.07 106.6) (width 0.25) (layer F.Cu) (net 7))
-  (segment (start 149.5311 106.1389) (end 149.5311 102.9936) (width 0.25) (layer F.Cu) (net 7))
-  (segment (start 149.07 106.6) (end 149.5311 106.1389) (width 0.25) (layer F.Cu) (net 7))
-  (segment (start 150.07 113.16) (end 150.07 106.6) (width 0.25) (layer F.Cu) (net 8))
-  (segment (start 151.0311 105.6389) (end 151.0311 100.9936) (width 0.25) (layer F.Cu) (net 8))
-  (segment (start 150.07 106.6) (end 151.0311 105.6389) (width 0.25) (layer F.Cu) (net 8))
-  (segment (start 151.07 113.16) (end 151.07 106.6) (width 0.25) (layer F.Cu) (net 9))
-  (segment (start 152.5311 105.1389) (end 152.5311 102.9936) (width 0.25) (layer F.Cu) (net 9))
-  (segment (start 151.07 106.6) (end 152.5311 105.1389) (width 0.25) (layer F.Cu) (net 9))
-  (segment (start 152.07 113.16) (end 152.07 106.6) (width 0.25) (layer F.Cu) (net 10))
-  (segment (start 154.0311 104.6389) (end 154.0311 100.9936) (width 0.25) (layer F.Cu) (net 10))
-  (segment (start 152.07 106.6) (end 154.0311 104.6389) (width 0.25) (layer F.Cu) (net 10))
-  (segment (start 153.07 113.16) (end 153.07 106.6) (width 0.25) (layer F.Cu) (net 11))
-  (segment (start 155.5311 104.1389) (end 155.5311 102.9936) (width 0.25) (layer F.Cu) (net 11))
-  (segment (start 153.07 106.6) (end 155.5311 104.1389) (width 0.25) (layer F.Cu) (net 11))
-  (segment (start 142.07 113.16) (end 142.07 106.6) (width 0.25) (layer F.Cu) (net 12))
-  (segment (start 139.0311 103.5611) (end 139.0311 100.9936) (width 0.25) (layer F.Cu) (net 12))
-  (segment (start 142.07 106.6) (end 139.0311 103.5611) (width 0.25) (layer F.Cu) (net 12))
-  (segment (start 142.06 113.13) (end 142.113 113.157) (width 0.25) (layer F.Cu) (net 12) (status 80000))
-  (segment (start 154.07 113.16) (end 154.07 106.6) (width 0.25) (layer F.Cu) (net 13))
-  (segment (start 156.97 103.7) (end 156.97 101.0547) (width 0.25) (layer F.Cu) (net 13))
-  (segment (start 154.07 106.6) (end 156.97 103.7) (width 0.25) (layer F.Cu) (net 13))
+  (segment (start 149.07 112.76) (end 149.07 106.5) (width 0.25) (layer F.Cu) (net 7) (status 400000))
+  (segment (start 149.5311 106.0389) (end 149.5311 102.9936) (width 0.25) (layer F.Cu) (net 7) (status 800000))
+  (segment (start 149.07 106.5) (end 149.5311 106.0389) (width 0.25) (layer F.Cu) (net 7))
+  (segment (start 150.07 112.76) (end 150.07 106.5) (width 0.25) (layer F.Cu) (net 8) (status 400000))
+  (segment (start 151.0311 105.5389) (end 151.0311 100.9936) (width 0.25) (layer F.Cu) (net 8) (status 800000))
+  (segment (start 150.07 106.5) (end 151.0311 105.5389) (width 0.25) (layer F.Cu) (net 8))
+  (segment (start 151.07 112.76) (end 151.07 106.5) (width 0.25) (layer F.Cu) (net 9) (status 400000))
+  (segment (start 152.5311 105.0389) (end 152.5311 102.9936) (width 0.25) (layer F.Cu) (net 9) (status 800000))
+  (segment (start 151.07 106.5) (end 152.5311 105.0389) (width 0.25) (layer F.Cu) (net 9))
+  (segment (start 152.07 112.76) (end 152.07 106.5) (width 0.25) (layer F.Cu) (net 10) (status 400000))
+  (segment (start 154.0311 104.5389) (end 154.0311 100.9936) (width 0.25) (layer F.Cu) (net 10) (status 800000))
+  (segment (start 152.07 106.5) (end 154.0311 104.5389) (width 0.25) (layer F.Cu) (net 10))
+  (segment (start 153.07 112.76) (end 153.07 106.5) (width 0.25) (layer F.Cu) (net 11) (status 400000))
+  (segment (start 155.5311 104.0389) (end 155.5311 102.9936) (width 0.25) (layer F.Cu) (net 11) (status 800000))
+  (segment (start 153.07 106.5) (end 155.5311 104.0389) (width 0.25) (layer F.Cu) (net 11))
+  (segment (start 142.07 112.76) (end 142.07 106.5) (width 0.25) (layer F.Cu) (net 12) (status 400000))
+  (segment (start 139.0311 103.4611) (end 139.0311 100.9936) (width 0.25) (layer F.Cu) (net 12) (status 800000))
+  (segment (start 142.07 106.5) (end 139.0311 103.4611) (width 0.25) (layer F.Cu) (net 12))
+  (segment (start 142.06 112.73) (end 142.113 112.757) (width 0.25) (layer F.Cu) (net 12) (status 80000))
+  (segment (start 154.07 112.76) (end 154.07 106.5) (width 0.25) (layer F.Cu) (net 13) (status 400000))
+  (segment (start 157.0311 103.5389) (end 157.0311 100.9936) (width 0.25) (layer F.Cu) (net 13) (status 800000))
+  (segment (start 154.07 106.5) (end 157.0311 103.5389) (width 0.25) (layer F.Cu) (net 13))
   (segment (start 156.97 101.0547) (end 157.0311 100.9936) (width 0.25) (layer F.Cu) (net 13))
-  (segment (start 141.07 113.16) (end 141.07 106.6) (width 0.25) (layer F.Cu) (net 14))
-  (segment (start 141.07 106.6) (end 137.5311 103.0611) (width 0.25) (layer F.Cu) (net 14))
+  (segment (start 141.07 112.76) (end 141.07 106.5) (width 0.25) (layer F.Cu) (net 14) (status 400000))
+  (segment (start 141.07 106.5) (end 137.5636 102.9936) (width 0.25) (layer F.Cu) (net 14) (status 800000))
+  (segment (start 137.5636 102.9936) (end 137.5311 102.9936) (width 0.25) (layer F.Cu) (net 14) (status C00000))
   (segment (start 137.5311 103.0611) (end 137.5311 102.9936) (width 0.25) (layer F.Cu) (net 14))
-  (segment (start 141.06 113.13) (end 141.097 113.157) (width 0.25) (layer F.Cu) (net 14) (status 80000))
-  (segment (start 155.07 113.16) (end 155.07 106.6) (width 0.25) (layer F.Cu) (net 15))
-  (segment (start 155.07 106.6) (end 158.5311 103.1389) (width 0.25) (layer F.Cu) (net 15))
+  (segment (start 141.06 112.73) (end 141.097 112.757) (width 0.25) (layer F.Cu) (net 14) (status 80000))
+  (segment (start 155.07 112.76) (end 155.07 106.6) (width 0.25) (layer F.Cu) (net 15) (status 400000))
+  (segment (start 155.07 106.6) (end 158.5311 103.1389) (width 0.25) (layer F.Cu) (net 15) (status 800000))
+  (segment (start 158.5311 103.1389) (end 158.5311 102.9936) (width 0.25) (layer F.Cu) (net 15) (status C00000))
   (segment (start 158.5311 103.1389) (end 158.5311 102.9936) (width 0.25) (layer F.Cu) (net 15))
 )

Commit message: Prace nad płytką
Parts:
- removed the ? at (148.0, 104.0)
- removed the ? at (148.0, 115.2)
- added ?: , Pin_Headers:Pin_Header_Straight_1x05_Pitch2.54mm, F.Cu at (158.7, 104.6)
- added ?: , objects:FFC_connector_15x1.0mm, F.Cu at (147.9, 113.8)
- added ?: , objects:flat_cable_connector_16pin, F.Cu at (148.3, 100.8)
Routing:
- net Net-(P1-Pad12): track 12.6 -> 0.00 mm
- net Net-(P1-Pad6): track 12.2 -> 0.00 mm
- net Net-(P1-Pad15): track 11.3 -> 0.00 mm
- net Net-(P1-Pad9): track 9.96 -> 0.00 mm
- net Net-(P1-Pad13): track 10.8 -> 20.0 mm
- net Net-(P2-Pad5): track 0.00 -> 8.82 mm
- net Net-(P2-Pad3): track 0.00 -> 8.22 mm
- net Net-(P2-Pad1): track 0.00 -> 6.80 mm
- net Net-(P2-Pad4): track 0.00 -> 6.46 mm
- net Net-(P1-Pad11): track 10.4 -> 16.3 mm
- net Net-(P1-Pad7): track 9.99 -> 15.7 mm
- net Net-(P1-Pad10): track 12.2 -> 17.8 mm
- net Net-(P1-Pad14): track 13.1 -> 18.6 mm
- net Net-(P2-Pad2): track 0.00 -> 5.27 mm
- net Net-(P1-Pad5): track 10.4 -> 12.8 mm
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Other:
- board size 25 x 25 mm -> 25 x 28.2 mm
